Commit message: Release UR5 pick-and-place dashboard v2.0
Add the local ROS dashboard, end-effector telemetry, experiment tooling, and tests.

Co-authored-by: Copilot <223556219+Copilot@users.noreply.github.com>

File: ur5_description/urdf/gazebo.xacro (robot description, xacro)
@@ -3,5 +3,5 @@
   <!-- IgnitionROS2Control plugin — loaded by gz_sim when the robot is spawned -->
   <gazebo>
-    <plugin filename="ign_ros2_control-system" name="ign_ros2_control::IgnitionROS2ControlPlugin">
+    <plugin filename="gz_ros2_control-system" name="gz_ros2_control::GazeboSimROS2ControlPlugin">
       <!-- Controller configuration used by the current bringup package. -->
       <parameters>$(find ur5_moveit_config)/config/ros2_controllers.yaml</parameters>

File: ur5_description/urdf/inc/ur_joint_control.xacro (robot description, xacro)
@@ -5,5 +5,5 @@
     Only position command + position/velocity state interfaces are declared.
     Velocity and effort command interfaces are removed: declaring interfaces
-    that no loaded controller claims causes IgnitionSystem to emit warnings on
+    that no loaded controller claims causes the GazeboSimSystem to emit warnings on
     every update cycle and can delay joint-state initialisation.
     If you later add a velocity or effort controller, re-add the corresponding

File: ur5_description/urdf/robotiq_gripper.ros2_control.xacro (robot description, xacro)
@@ -32,5 +32,5 @@
                 </xacro:if>
                 <xacro:if value="${sim_ignition}">
-                    <plugin>ign_ros2_control/IgnitionSystem</plugin>
+                    <plugin>gz_ros2_control/GazeboSimSystem</plugin>
                 </xacro:if>
                 <xacro:if value="${use_fake_hardware}">
@@ -54,5 +54,8 @@
                 <command_interface name="position" />
                 <state_interface name="position">
-                    <param name="initial_value">${gripper_closed_position}</param>
+                    <!-- Ignition's passive mimic joints spawn at zero. Start
+                         the driver open too, so the linkage is assembled before
+                         the velocity-based mimic controller begins updating. -->
+                    <param name="initial_value">${0.0 if sim_ignition else gripper_closed_position}</param>
                 </state_interface>
                 <state_interface name="velocity"/>

File: ur5_description/urdf/robotiq_gripper_macro.xacro (robot description, xacro)
@@ -20,4 +20,9 @@
         gripper_max_force:=235.0
         gripper_closed_position:=0.7929">
+        <!-- Keep commanded endpoints (0 and 0.8 rad) just inside Gazebo's
+             physical stops. Its velocity-driven knuckles can stick at an exact
+             stop, breaking synchronization with the continuous mimic joints.
+             MoveIt retains the nominal 0..0.8 range in joint_limits.yaml. -->
+        <xacro:property name="knuckle_stop_margin" value="${0.001 if sim_ignition else 0.0}" />
         <!-- ros2 control include -->
         <xacro:include filename="$(find ur5_description)/urdf/robotiq_gripper.ros2_control.xacro" />
@@ -257,5 +262,5 @@
             <axis xyz="0 -1 0" />
             <origin xyz="0.03060114 0.0 0.05490452" rpy="0 0 0" />
-            <limit lower="0.0" upper="0.8" velocity="0.5" effort="50" />
+            <limit lower="${-knuckle_stop_margin}" upper="${0.8 + knuckle_stop_margin}" velocity="0.5" effort="50" />
         </joint>
         <joint name="${prefix}robotiq_85_right_knuckle_joint" type="revolute">
@@ -264,5 +269,5 @@
             <axis xyz="0 -1 0" />
             <origin xyz="-0.03060114 0.0 0.05490452" rpy="0 0 0" />
-            <limit lower="-0.8" upper="0.0" velocity="0.5" effort="50" />
+            <limit lower="${-0.8 - knuckle_stop_margin}" upper="${knuckle_stop_margin}" velocity="0.5" effort="50" />
             <mimic joint="${prefix}robotiq_85_left_knuckle_joint" multiplier="-1" />
         </joint>

File: ur5_description/urdf/ur5_with_gripper.urdf.xacro (robot description, xacro)
@@ -139,5 +139,5 @@
     </gazebo>
     <gazebo>
-      <plugin filename="ign_ros2_control-system" name="ign_ros2_control::IgnitionROS2ControlPlugin">
+      <plugin filename="gz_ros2_control-system" name="gz_ros2_control::GazeboSimROS2ControlPlugin">
         <parameters>$(arg simulation_controllers)</parameters>
         <controller_manager_node_name>$(arg tf_prefix)controller_manager</controller_manager_node_name>

File: ur5_moveit_config/config/ur5.ros2_control.xacro (robot description, xacro)
@@ -6,5 +6,5 @@
             <hardware>
                 <xacro:if value="${use_sim == 'true' or use_sim == True or use_sim == '1'}">
-                    <plugin>ign_ros2_control/IgnitionSystem</plugin>
+                    <plugin>gz_ros2_control/GazeboSimSystem</plugin>
                 </xacro:if>
                 <xacro:unless value="${use_sim == 'true' or use_sim == True or use_sim == '1'}">
@@ -90,5 +90,5 @@
         <xacro:if value="${use_sim == 'true' or use_sim == True or use_sim == '1'}">
             <gazebo>
-                <plugin filename="ign_ros2_control-system" name="ign_ros2_control::IgnitionROS2ControlPlugin">
+                <plugin filename="gz_ros2_control-system" name="gz_ros2_control::GazeboSimROS2ControlPlugin">
                     <parameters>$(find ur5_moveit_config)/config/ros2_controllers.yaml</parameters>
                 </plugin>

File: ur5_moveit_config/config/ur5.urdf.xacro (robot description, xacro)
@@ -151,5 +151,5 @@
     </gazebo>
     <gazebo>
-      <plugin filename="ign_ros2_control-system" name="ign_ros2_control::IgnitionROS2ControlPlugin">
+      <plugin filename="gz_ros2_control-system" name="gz_ros2_control::GazeboSimROS2ControlPlugin">
         <parameters>$(arg simulation_controllers)</parameters>
         <controller_manager_node_name>$(arg tf_prefix)controller_manager</controller_manager_node_name>
