Commit message: Release fixed PID gains and tuning data

File: ur5_description/urdf/ur5.ros2_control.xacro (robot description, xacro)
@@ -21,4 +21,5 @@
     non_blocking_read:=true
     keep_alive_count:=2
+    controller_mode:=position
     ">
     <ros2_control name="${name}" type="system">
@@ -68,4 +69,7 @@
         <command_interface name="position"/>
         <command_interface name="velocity"/>
+        <xacro:if value="${controller_mode == 'effort'}">
+          <command_interface name="effort"/>
+        </xacro:if>
         <state_interface name="position">
           <!-- initial position for the FakeSystem and simulation -->
@@ -73,9 +77,14 @@
         </state_interface>
         <state_interface name="velocity"/>
-        <state_interface name="effort"/>
+        <state_interface name="effort">
+          <param name="initial_value">0.0</param>
+        </state_interface>
       </joint>
       <joint name="${tf_prefix}shoulder_lift_joint">
         <command_interface name="position"/>
         <command_interface name="velocity"/>
+        <xacro:if value="${controller_mode == 'effort'}">
+          <command_interface name="effort"/>
+        </xacro:if>
         <state_interface name="position">
           <!-- initial position for the FakeSystem and simulation -->
@@ -83,9 +92,14 @@
         </state_interface>
         <state_interface name="velocity"/>
-        <state_interface name="effort"/>
+        <state_interface name="effort">
+          <param name="initial_value">-1.40716</param>
+        </state_interface>
       </joint>
       <joint name="${tf_prefix}elbow_joint">
         <command_interface name="position"/>
         <command_interface name="velocity"/>
+        <xacro:if value="${controller_mode == 'effort'}">
+          <command_interface name="effort"/>
+        </xacro:if>
         <state_interface name="position">
           <!-- initial position for the FakeSystem and simulation -->
@@ -93,9 +107,14 @@
         </state_interface>
         <state_interface name="velocity"/>
-        <state_interface name="effort"/>
+        <state_interface name="effort">
+          <param name="initial_value">0.2707</param>
+        </state_interface>
       </joint>
       <joint name="${tf_prefix}wrist_1_joint">
         <command_interface name="position"/>
         <command_interface name="velocity"/>
+        <xacro:if value="${controller_mode == 'effort'}">
+          <command_interface name="effort"/>
+        </xacro:if>
         <state_interface name="position">
           <!-- initial position for the FakeSystem and simulation -->
@@ -103,9 +122,14 @@
         </state_interface>
         <state_interface name="velocity"/>
-        <state_interface name="effort"/>
+        <state_interface name="effort">
+          <param name="initial_value">-0.0553</param>
+        </state_interface>
       </joint>
       <joint name="${tf_prefix}wrist_2_joint">
         <command_interface name="position"/>
         <command_interface name="velocity"/>
+        <xacro:if value="${controller_mode == 'effort'}">
+          <command_interface name="effort"/>
+        </xacro:if>
         <state_interface name="position">
           <!-- initial position for the FakeSystem and simulation -->
@@ -113,9 +137,14 @@
         </state_interface>
         <state_interface name="velocity"/>
-        <state_interface name="effort"/>
+        <state_interface name="effort">
+          <param name="initial_value">0.1036</param>
+        </state_interface>
       </joint>
       <joint name="${tf_prefix}wrist_3_joint">
         <command_interface name="position"/>
         <command_interface name="velocity"/>
+        <xacro:if value="${controller_mode == 'effort'}">
+          <command_interface name="effort"/>
+        </xacro:if>
         <state_interface name="position">
           <!-- initial position for the FakeSystem and simulation -->
@@ -123,5 +152,7 @@
         </state_interface>
         <state_interface name="velocity"/>
-        <state_interface name="effort"/>
+        <state_interface name="effort">
+          <param name="initial_value">0.0</param>
+        </state_interface>
       </joint>
       <xacro:unless value="${sim_gazebo or sim_ignition}">

File: ur5_description/urdf/ur5_macro.xacro (robot description, xacro)
@@ -42,5 +42,6 @@
     trajectory_port:=50003
     non_blocking_read:=true
-    keep_alive_count:=2"
+    keep_alive_count:=2
+    controller_mode:=position"
     >
     <!-- Load configuration data from the provided .yaml files -->
@@ -63,4 +64,5 @@
         sim_gazebo="${sim_gazebo}"
         sim_ignition="${sim_ignition}"
+        controller_mode="${controller_mode}"
         script_filename="${script_filename}"
         output_recipe_filename="${output_recipe_filename}"
@@ -300,5 +302,5 @@
          <safety_controller soft_lower_limit="${shoulder_pan_lower_limit + safety_pos_margin}" soft_upper_limit="${shoulder_pan_upper_limit - safety_pos_margin}" k_position="${safety_k_position}" k_velocity="0.0"/>
       </xacro:if>
-      <dynamics damping="0" friction="0"/>
+      <dynamics damping="0.1" friction="0"/>
     </joint>
     <joint name="${tf_prefix}shoulder_lift_joint" type="revolute">
@@ -312,5 +314,5 @@
          <safety_controller soft_lower_limit="${shoulder_lift_lower_limit + safety_pos_margin}" soft_upper_limit="${shoulder_lift_upper_limit - safety_pos_margin}" k_position="${safety_k_position}" k_velocity="0.0"/>
       </xacro:if>
-      <dynamics damping="0" friction="0"/>
+      <dynamics damping="0.1" friction="0"/>
     </joint>
     <joint name="${tf_prefix}elbow_joint" type="revolute">
@@ -324,5 +326,5 @@
          <safety_controller soft_lower_limit="${elbow_joint_lower_limit + safety_pos_margin}" soft_upper_limit="${elbow_joint_upper_limit - safety_pos_margin}" k_position="${safety_k_position}" k_velocity="0.0"/>
       </xacro:if>
-      <dynamics damping="0" friction="0"/>
+      <dynamics damping="0.1" friction="0"/>
     </joint>
     <joint name="${tf_prefix}wrist_1_joint" type="revolute">
@@ -336,5 +338,5 @@
          <safety_controller soft_lower_limit="${wrist_1_lower_limit + safety_pos_margin}" soft_upper_limit="${wrist_1_upper_limit - safety_pos_margin}" k_position="${safety_k_position}" k_velocity="0.0"/>
       </xacro:if>
-      <dynamics damping="0" friction="0"/>
+      <dynamics damping="0.1" friction="0"/>
     </joint>
     <joint name="${tf_prefix}wrist_2_joint" type="revolute">
@@ -348,5 +350,5 @@
          <safety_controller soft_lower_limit="${wrist_2_lower_limit + safety_pos_margin}" soft_upper_limit="${wrist_2_upper_limit - safety_pos_margin}" k_position="${safety_k_position}" k_velocity="0.0"/>
       </xacro:if>
-      <dynamics damping="0" friction="0"/>
+      <dynamics damping="0.1" friction="0"/>
     </joint>
     <joint name="${tf_prefix}wrist_3_joint" type="${wrist_3_joint_type}">
@@ -368,5 +370,5 @@
         </xacro:if>
       </xacro:unless>
-      <dynamics damping="0" friction="0"/>
+      <dynamics damping="0.5" friction="0"/>
     </joint>
     <link name="${tf_prefix}ft_frame"/>

File: ur5_description/urdf/ur_macro.xacro (robot description, xacro)
@@ -190,5 +190,5 @@
         <safety_controller soft_lower_limit="${shoulder_lift_lower_limit + safety_pos_margin}" soft_upper_limit="${shoulder_lift_upper_limit - safety_pos_margin}" k_position="${safety_k_position}" k_velocity="0.0"/>
       </xacro:if>
-      <dynamics damping="100.0" friction="0.1"/>
+      <dynamics damping="100.0" friction="3.0"/>
     </joint>
     <joint name="${tf_prefix}elbow_joint" type="revolute">
@@ -201,5 +201,5 @@
         <safety_controller soft_lower_limit="${elbow_joint_lower_limit + safety_pos_margin}" soft_upper_limit="${elbow_joint_upper_limit - safety_pos_margin}" k_position="${safety_k_position}" k_velocity="0.0"/>
       </xacro:if>
-      <dynamics damping="100.0" friction="0.1"/>
+      <dynamics damping="100.0" friction="1.0"/>
     </joint>
     <joint name="${tf_prefix}wrist_1_joint" type="revolute">
@@ -212,5 +212,5 @@
         <safety_controller soft_lower_limit="${wrist_1_lower_limit + safety_pos_margin}" soft_upper_limit="${wrist_1_upper_limit - safety_pos_margin}" k_position="${safety_k_position}" k_velocity="0.0"/>
       </xacro:if>
-      <dynamics damping="10.0" friction="0.1"/>
+      <dynamics damping="10.0" friction="0.5"/>
     </joint>
     <joint name="${tf_prefix}wrist_2_joint" type="revolute">
@@ -223,5 +223,5 @@
         <safety_controller soft_lower_limit="${wrist_2_lower_limit + safety_pos_margin}" soft_upper_limit="${wrist_2_upper_limit - safety_pos_margin}" k_position="${safety_k_position}" k_velocity="0.0"/>
       </xacro:if>
-      <dynamics damping="10.0" friction="0.1"/>
+      <dynamics damping="10.0" friction="0.5"/>
     </joint>
     <joint name="${tf_prefix}wrist_3_joint" type="${wrist_3_joint_type}">

File: ur5_moveit_config/config/ur5.urdf.xacro (robot description, xacro)
@@ -46,4 +46,5 @@
    <xacro:arg name="simulation_controllers" default="" />
    <xacro:arg name="simulated_grasp" default="false" />
+   <xacro:arg name="controller_mode" default="position" />
    <!-- <xacro:arg name="simulation_controllers" default="$(find-pkg-share ur_yt_sim)/config/ur5_controllers_gripper.yaml" /> -->
    <!-- initial position for simulations (Fake Hardware, Gazebo, Ignition) -->
@@ -117,4 +118,5 @@
      script_sender_port="$(arg script_sender_port)"
      trajectory_port="$(arg trajectory_port)"
+     controller_mode="$(arg controller_mode)"
      >
      <origin xyz="1.10 0 0.34" rpy="0 0 1.5707963267948966" />
@@ -150,4 +152,41 @@
     <gazebo reference="world">
     </gazebo>
+    <!-- Joint force/torque sensors for DART transmitted wrench evaluation -->
+    <gazebo reference="$(arg tf_prefix)shoulder_pan_joint">
+      <sensor name="$(arg tf_prefix)shoulder_pan_ft" type="force_torque">
+        <always_on>true</always_on>
+        <update_rate>1000</update_rate>
+      </sensor>
+    </gazebo>
+    <gazebo reference="$(arg tf_prefix)shoulder_lift_joint">
+      <sensor name="$(arg tf_prefix)shoulder_lift_ft" type="force_torque">
+        <always_on>true</always_on>
+        <update_rate>1000</update_rate>
+      </sensor>
+    </gazebo>
+    <gazebo reference="$(arg tf_prefix)elbow_joint">
+      <sensor name="$(arg tf_prefix)elbow_joint_ft" type="force_torque">
+        <always_on>true</always_on>
+        <update_rate>1000</update_rate>
+      </sensor>
+    </gazebo>
+    <gazebo reference="$(arg tf_prefix)wrist_1_joint">
+      <sensor name="$(arg tf_prefix)wrist_1_ft" type="force_torque">
+        <always_on>true</always_on>
+        <update_rate>1000</update_rate>
+      </sensor>
+    </gazebo>
+    <gazebo reference="$(arg tf_prefix)wrist_2_joint">
+      <sensor name="$(arg tf_prefix)wrist_2_ft" type="force_torque">
+        <always_on>true</always_on>
+        <update_rate>1000</update_rate>
+      </sensor>
+    </gazebo>
+    <gazebo reference="$(arg tf_prefix)wrist_3_joint">
+      <sensor name="$(arg tf_prefix)wrist_3_ft" type="force_torque">
+        <always_on>true</always_on>
+        <update_rate>1000</update_rate>
+      </sensor>
+    </gazebo>
     <gazebo>
       <plugin filename="gz_ros2_control-system" name="gz_ros2_control::GazeboSimROS2ControlPlugin">
