Commit message: feat: save current workspace state
Co-authored-by: Copilot <223556219+Copilot@users.noreply.github.com>

File: ur5_description/urdf/robotiq_gripper_macro.xacro (robot description, xacro)
@@ -185,5 +185,5 @@
                 </geometry>
             </visual>
-            <collision>
+            <collision name="${prefix}robotiq_85_left_finger_tip_link_collision">
                 <geometry>
                     <!-- <mesh filename="package://robotiq_description/meshes/collision/2f_85/left_finger_tip.stl" /> -->
@@ -222,5 +222,5 @@
                 </geometry>
             </visual>
-            <collision>
+            <collision name="${prefix}robotiq_85_right_finger_tip_link_collision">
                 <geometry>
                     <!-- <mesh filename="package://robotiq_description/meshes/collision/2f_85/right_finger_tip.stl" /> -->

File: ur5_moveit_config/config/ur5.urdf.xacro (robot description, xacro)
@@ -187,4 +187,25 @@
         <always_on>true</always_on>
         <update_rate>1000</update_rate>
+        <topic>/wrist_ft/wrench</topic>
+      </sensor>
+    </gazebo>
+    <gazebo reference="$(arg tf_prefix)robotiq_85_left_finger_tip_link">
+      <sensor name="$(arg tf_prefix)left_fingertip_contact" type="contact">
+        <contact>
+          <collision>$(arg tf_prefix)robotiq_85_left_finger_tip_link_collision</collision>
+        </contact>
+        <always_on>true</always_on>
+        <update_rate>100</update_rate>
+        <topic>/fingertip/left_contact</topic>
+      </sensor>
+    </gazebo>
+    <gazebo reference="$(arg tf_prefix)robotiq_85_right_finger_tip_link">
+      <sensor name="$(arg tf_prefix)right_fingertip_contact" type="contact">
+        <contact>
+          <collision>$(arg tf_prefix)robotiq_85_right_finger_tip_link_collision</collision>
+        </contact>
+        <always_on>true</always_on>
+        <update_rate>100</update_rate>
+        <topic>/fingertip/right_contact</topic>
       </sensor>
     </gazebo>
